Commit message: refactor URDF and launch file for multi-robot support

File: robot_description/urdf/robot.xacro (robot description, xacro)
@@ -1,15 +1,49 @@
 <?xml version="1.0"?>
-<robot name="robot" xmlns:xacro="http://ros.org/wiki/xacro">
-<!-- ===============================================================
-                            [LINKS]
-================================================================ -->
-    <!-- ─────────────────────────────────────────────
-        [LINKS] BASE FOOTPRINT
-    ────────────────────────────────────────────── -->
-    <link name="base_footprint"/>
-    <!-- ─────────────────────────────────────────────
-        [LINKS] BASE LINK
-    ────────────────────────────────────────────── -->
-    <link name="base_link">
+<robot name="robot" xmlns:xacro="http://www.ros.org/wiki/xacro">
+    <!-- **********************************************************************
+        [PROPERTIES]
+    *********************************************************************** -->
+    <xacro:property name="PI"           value="3.14159265"/>
+    <xacro:property name="mesh_dir"     value="package://robot_description/meshes"/>
+    <!-- **********************************************************************
+        [ARG]
+    *********************************************************************** -->
+    <xacro:arg name="ns"                default="r1"/>
+    <!-- **********************************************************************
+        [CUSTOM COLOR]
+    *********************************************************************** -->
+    <material name="base_color">
+        <color rgba="0.52 0.55 0.81 1.0"/>
+    </material>
+    <material name="wheel_color">
+        <color rgba="0.15 0.15 0.15 1.0"/>
+    </material>
+    <material name="lidar_color">
+        <color rgba="0.93 0.91 0.17 1.0"/>
+    </material>
+    <!-- **********************************************************************
+        [LINKS]
+    *********************************************************************** -->
+    <!-- ───────────────────────────────────────────────────────────────────────
+        [LINKS] Base Footprint
+    ──────────────────────────────────────────────────────────────────────── -->
+    <link name="$(arg ns)_base_footprint"/>
+    <!-- ───────────────────────────────────────────────────────────────────────
+        [LINKS] Base Link
+    ──────────────────────────────────────────────────────────────────────── -->
+    <link name="$(arg ns)_base_link">
+        <visual>
+            <origin xyz="0.0 0.0 0.0" rpy="0.0 0.0 0.0"/>
+            <geometry>
+                <mesh filename="${mesh_dir}/base_link.STL" scale="1 1 1"/>
+            </geometry>
+            <material name="base_color"/>
+        </visual>
+        <collision>
+            <origin xyz="0.0 0.0 0.0" rpy="0.0 0.0 0.0"/>
+            <geometry>
+                <mesh filename="${mesh_dir}/base_link.STL" scale="1 1 1"/>
+            </geometry>
+        </collision>
         <inertial>
             <origin xyz="0.049 -0.002 0.219" rpy="0.0 0.0 0.0"/>
@@ -18,24 +52,22 @@
                     iyy="0.089" iyz="4.051E-07" izz="0.059"/>
         </inertial>
-        <visual>
-            <origin xyz="0.0 0.0 0.0" rpy="0.0 0.0 0.0"/>
-            <geometry>
-                <mesh filename="package://robot_description/meshes/base_link.STL" scale="1 1 1"/>
-            </geometry>
-            <material name="material_base_link">
-                <color rgba="0.52 0.55 0.81 1.0"/>
-            </material>
+    </link>
+    <!-- ───────────────────────────────────────────────────────────────────────
+        [LINKS] Wheel Left
+    ──────────────────────────────────────────────────────────────────────── -->
+    <link name="$(arg ns)_wheel_left_link">
+        <visual>
+            <origin xyz="0.0 0.0 0.0" rpy="0.0 0.0 0.0"/>
+            <geometry>
+                <mesh filename="${mesh_dir}/wheel_left.STL" scale="1 1 1"/>
+            </geometry>
+            <material name="wheel_color"/>
         </visual>
         <collision>
             <origin xyz="0.0 0.0 0.0" rpy="0.0 0.0 0.0"/>
             <geometry>
-                <mesh filename="package://robot_description/meshes/base_link.STL" scale="1 1 1"/>
+                <mesh filename="${mesh_dir}/wheel_left.STL" scale="1 1 1"/>
             </geometry>
         </collision>
-    </link>
-    <!-- ─────────────────────────────────────────────
-        [LINKS] WHEEL LEFT
-    ────────────────────────────────────────────── -->
-    <link name="wheel_left_link">
         <inertial>
             <origin xyz="-0.014 0.001 -0.033" rpy="0.0 0.0 0.0"/>
@@ -44,24 +76,22 @@
                     iyy="0.002" iyz="4.986E-20" izz="0.001"/>
         </inertial>
-        <visual>
-            <origin xyz="0.0 0.0 0.0" rpy="0.0 0.0 0.0"/>
-            <geometry>
-                <mesh filename="package://robot_description/meshes/wheel_left.STL" scale="1 1 1"/>
-            </geometry>
-            <material name="material_wheel_left">
-                <color rgba="0.15 0.15 0.15 1.0"/>
-            </material>
+    </link>
+    <!-- ───────────────────────────────────────────────────────────────────────
+        [LINKS] Wheel Right
+    ──────────────────────────────────────────────────────────────────────── -->
+    <link name="$(arg ns)_wheel_right_link">
+        <visual>
+            <origin xyz="0.0 0.0 0.0" rpy="0.0 0.0 0.0"/>
+            <geometry>
+                <mesh filename="${mesh_dir}/wheel_right.STL" scale="1 1 1"/>
+            </geometry>
+            <material name="wheel_color"/>
         </visual>
         <collision>
             <origin xyz="0.0 0.0 0.0" rpy="0.0 0.0 0.0"/>
             <geometry>
-                <mesh filename="package://robot_description/meshes/wheel_left.STL" scale="1 1 1"/>
+                <mesh filename="${mesh_dir}/wheel_right.STL" scale="1 1 1"/>
             </geometry>
         </collision>
-    </link>
-    <!-- ─────────────────────────────────────────────
-        [LINKS] WHEEL RIGHT
-    ────────────────────────────────────────────── -->
-    <link name="wheel_right_link">
         <inertial>
             <origin xyz="-0.014 0.001 -0.033" rpy="0.0 0.0 0.0"/>
@@ -70,24 +100,22 @@
                      iyy="0.002" iyz="2.955E-22" izz="0.001"/>
         </inertial>
-        <visual>
-            <origin xyz="0.0 0.0 0.0" rpy="0.0 0.0 0.0"/>
-            <geometry>
-                <mesh filename="package://robot_description/meshes/wheel_right.STL" scale="1 1 1"/>
-            </geometry>
-            <material name="material_wheel_right">
-                <color rgba="0.15 0.15 0.15 1.0"/>
-            </material>
+    </link>
+    <!-- ───────────────────────────────────────────────────────────────────────
+        [LINKS] Caster Left
+    ──────────────────────────────────────────────────────────────────────── -->
+    <link name="$(arg ns)_caster_left_link">
+        <visual>
+            <origin xyz="0.0 0.0 0.0" rpy="0.0 0.0 0.0"/>
+            <geometry>
+                <mesh filename="${mesh_dir}/caster_left.STL" scale="1 1 1"/>
+            </geometry>
+            <material name="wheel_color"/>
         </visual>
         <collision>
             <origin xyz="0.0 0.0 0.0" rpy="0.0 0.0 0.0"/>
             <geometry>
-                <mesh filename="package://robot_description/meshes/wheel_right.STL" scale="1 1 1"/>
+                <mesh filename="${mesh_dir}/caster_left.STL" scale="1 1 1"/>
             </geometry>
         </collision>
-    </link>
-    <!-- ─────────────────────────────────────────────
-        [LINKS] CASTER LEFT
-    ────────────────────────────────────────────── -->
-    <link name="caster_left_link">
         <inertial>
             <origin xyz="-0.014 0.001 -0.033" rpy="0.0 0.0 0.0"/>
@@ -96,24 +124,22 @@
                     iyy="2.851E-05" iyz="3.766E-07" izz="2.982E-05"/>
         </inertial>
-        <visual>
-            <origin xyz="0.0 0.0 0.0" rpy="0.0 0.0 0.0"/>
-            <geometry>
-                <mesh filename="package://robot_description/meshes/caster_left.STL" scale="1 1 1"/>
-            </geometry>
-            <material name="material_caster_left">
-                <color rgba="0.15 0.15 0.15 1.0"/>
-            </material>
+    </link>
+    <!-- ───────────────────────────────────────────────────────────────────────
+        [LINKS] Caster Right
+    ──────────────────────────────────────────────────────────────────────── -->
+    <link name="$(arg ns)_caster_right_link">
+        <visual>
+            <origin xyz="0.0 0.0 0.0" rpy="0.0 0.0 0.0"/>
+            <geometry>
+                <mesh filename="${mesh_dir}/caster_right.STL" scale="1 1 1"/>
+            </geometry>
+            <material name="wheel_color"/>
         </visual>
         <collision>
             <origin xyz="0.0 0.0 0.0" rpy="0.0 0.0 0.0"/>
             <geometry>
-                <mesh filename="package://robot_description/meshes/caster_left.STL" scale="1 1 1"/>
+                <mesh filename="${mesh_dir}/caster_right.STL" scale="1 1 1"/>
             </geometry>
         </collision>
-    </link>
-    <!-- ─────────────────────────────────────────────
-        [LINKS] CASTER RIGHT
-    ────────────────────────────────────────────── -->
-    <link name="caster_right_link">
         <inertial>
             <origin xyz="-0.014 0.001 -0.033" rpy="0.0 0.0 0.0"/>
@@ -122,133 +148,116 @@
                     iyy="2.851E-05" iyz="3.766E-07" izz="2.982E-05"/>
         </inertial>
-        <visual>
-            <origin xyz="0.0 0.0 0.0" rpy="0.0 0.0 0.0"/>
-            <geometry>
-                <mesh filename="package://robot_description/meshes/caster_right.STL" scale="1 1 1"/>
-            </geometry>
-            <material name="material_caster_right">
-                <color rgba="0.15 0.15 0.15 1.0"/>
-            </material>
-        </visual>
-        <collision>
-            <origin xyz="0.0 0.0 0.0" rpy="0.0 0.0 0.0"/>
-            <geometry>
-                <mesh filename="package://robot_description/meshes/caster_right.STL" scale="1 1 1"/>
-            </geometry>
-        </collision>
-    </link>
-    <!-- ─────────────────────────────────────────────
-        [LINKS] IMU
-    ────────────────────────────────────────────── -->
-    <link name="imu_link"/>
-    <!-- ─────────────────────────────────────────────
-        [LINKS] LIDAR
-    ────────────────────────────────────────────── -->
-      <link name="lidar_link">
+    </link>
+    <!-- ───────────────────────────────────────────────────────────────────────
+        [LINKS] Imu
+    ──────────────────────────────────────────────────────────────────────── -->
+    <link name="$(arg ns)_imu_link"/>
+    <!-- ───────────────────────────────────────────────────────────────────────
+        [LINKS] Lidar
+    ──────────────────────────────────────────────────────────────────────── -->
+    <link name="$(arg ns)_lidar_link">
+        <visual>
+            <origin xyz="0 0 -0.05" rpy="0 0 0"/>
+            <geometry>
+                <mesh filename="${mesh_dir}/lidar_hokuyo_ust10.stl" scale="1 1 1"/>
+            </geometry>
+            <material name="lidar_color"/>
+        </visual>
+    </link>
+    <!-- ───────────────────────────────────────────────────────────────────────
+        [LINKS] Camera
+    ──────────────────────────────────────────────────────────────────────── -->
+    <link name="$(arg ns)_camera_link">
         <visual>
             <origin xyz="0 0 0" rpy="0 0 0"/>
             <geometry>
-                <mesh filename="package://robot_description/meshes/lidar_hokuyo_ust10.stl" scale="1 1 1"/>
-            </geometry>
-            <material name="material_lidar">
-                <color rgba="0.93 0.91 0.17 1.0"/>
-            </material>
-        </visual>
-    </link>
-    <!-- ─────────────────────────────────────────────
-        [LINKS] CAMERA DEPTH
-    ────────────────────────────────────────────── -->
-      <link name="camera_link">
-        <visual>
-            <origin xyz="0 0 0" rpy="0 0 0"/>
-            <geometry>
-                <mesh filename="package://robot_description/meshes/d435.dae" scale="1.1 1.1 1.1"/>
-            </geometry>
-        </visual>
-    </link>
-<!-- ===============================================================
-                            [JOINTS]
-================================================================ -->
-    <!-- ─────────────────────────────────────────────
-        [JOINTS] BASE
-    ────────────────────────────────────────────── -->
-    <joint name="base_joint" type="fixed">
+                <mesh filename="${mesh_dir}/d435.dae" scale="1.1 1.1 1.1"/>
+            </geometry>
+        </visual>
+    </link>
+    <!-- **********************************************************************
+        [JOINTS]
+    *********************************************************************** -->
+    <!-- ───────────────────────────────────────────────────────────────────────
+        [JOINTS] Base
+    ──────────────────────────────────────────────────────────────────────── -->
+    <joint name="$(arg ns)_base_joint" type="fixed">
         <origin xyz="0.0 0.0 0.035" rpy="0.0 0.0 0.0"/>
-        <parent link="base_footprint"/>
-        <child link="base_link"/>
-    </joint>
-    <!-- ─────────────────────────────────────────────
-        [JOINTS] WHEEL LEFT
-    ────────────────────────────────────────────── -->
-    <joint name="wheel_left_joint" type="continuous">
+        <parent link="$(arg ns)_base_footprint"/>
+        <child link="$(arg ns)_base_link"/>
+    </joint>
+    <!-- ───────────────────────────────────────────────────────────────────────
+        [JOINTS] Wheel Left
+    ──────────────────────────────────────────────────────────────────────── -->
+    <joint name="$(arg ns)_wheel_left_joint" type="continuous">
         <origin xyz="0.155 0.144 0.044" rpy="0.0 0.0 0.0"/>
-        <parent link="base_link"/>
-        <child link="wheel_left_link"/>
+        <parent link="$(arg ns)_base_link"/>
+        <child link="$(arg ns)_wheel_left_link"/>
         <axis xyz="0 1 0"/>
         <limit effort="10.0" velocity="10.0"/>
     </joint>
-    <!-- ─────────────────────────────────────────────
-        [JOINTS] WHEEL RIGHT
-    ────────────────────────────────────────────── -->
-    <joint name="wheel_right_joint" type="continuous">
+    <!-- ───────────────────────────────────────────────────────────────────────
+        [JOINTS] Wheel Right
+    ──────────────────────────────────────────────────────────────────────── -->
+    <joint name="$(arg ns)_wheel_right_joint" type="continuous">
         <origin xyz="0.155 -0.144 0.044" rpy="0.0 0.0 0.0"/>
-        <parent link="base_link"/>
-        <child link="wheel_right_link"/>
+        <parent link="$(arg ns)_base_link"/>
+        <child link="$(arg ns)_wheel_right_link"/>
         <axis xyz="0 1 0"/>
         <limit effort="10.0" velocity="10.0"/>
     </joint>
-    <!-- ─────────────────────────────────────────────
-        [JOINTS] CASTER LEFT
-    ────────────────────────────────────────────── -->
-    <joint name="caster_left_joint" type="fixed">
+    <!-- ───────────────────────────────────────────────────────────────────────
+        [JOINTS] Caster Left
+    ──────────────────────────────────────────────────────────────────────── -->
+    <joint name="$(arg ns)_caster_left_joint" type="fixed">
         <origin xyz="-0.1 0.085 0.038" rpy="0.0 0.0 0.0"/>
-        <parent link="base_link"/>
-        <child link="caster_left_link"/>
-    </joint>
-    <!-- ─────────────────────────────────────────────
-        [JOINTS] CASTER RIGHT
-    ────────────────────────────────────────────── -->
-    <joint name="caster_right_joint" type="fixed">
+        <parent link="$(arg ns)_base_link"/>
+        <child link="$(arg ns)_caster_left_link"/>
+    </joint>
+    <!-- ───────────────────────────────────────────────────────────────────────
+        [JOINTS] Caster Right
+    ──────────────────────────────────────────────────────────────────────── -->
+    <joint name="$(arg ns)_caster_right_joint" type="fixed">
         <origin xyz="-0.1 -0.085 0.038" rpy="0.0 0.0 0.0"/>
-        <parent link="base_link"/>
-        <child link="caster_right_link"/>
-    </joint>
-    <!-- ─────────────────────────────────────────────
-        [JOINTS] IMU
-    ────────────────────────────────────────────── -->
-    <joint name="imu_joint" type="fixed">
+        <parent link="$(arg ns)_base_link"/>
+        <child link="$(arg ns)_caster_right_link"/>
+    </joint>
+    <!-- ───────────────────────────────────────────────────────────────────────
+        [JOINTS] Imu
+    ──────────────────────────────────────────────────────────────────────── -->
+    <joint name="$(arg ns)_imu_joint" type="fixed">
         <origin xyz="0.0 0.0 0.0" rpy="0 0 0"/>
-        <parent link="base_link"/>
-        <child link="imu_link"/>
-    </joint>
-    <!-- ─────────────────────────────────────────────
-        [JOINTS] LIDAR
-    ────────────────────────────────────────────── -->
-    <joint name="lidar_joint" type="fixed">
-        <parent link="base_link"/>
-        <child link="lidar_link"/>
-        <origin xyz="0.318 0 0.084" rpy="0 0 0"/>
-    </joint>
-    <!-- ─────────────────────────────────────────────
-        [JOINTS] CAMERA DEPTH
-    ────────────────────────────────────────────── -->
-    <joint name="camera_joint" type="fixed">
-        <parent link="base_link"/>
-        <child link="camera_link"/>
+        <parent link="$(arg ns)_base_link"/>
+        <child link="$(arg ns)_imu_link"/>
+    </joint>
+    <!-- ───────────────────────────────────────────────────────────────────────
+        [JOINTS] Lidar
+    ──────────────────────────────────────────────────────────────────────── -->
+    <joint name="$(arg ns)_lidar_joint" type="fixed">
+        <origin xyz="0.318 0 0.134" rpy="0 0 0"/>
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